File: KiCAD/Taupunktlueftung.kicad_sch (KiCad schematic)
At the start: 29 parts, among them J1 DC in, J2 Micro_SD_Card_Adapter, J3 Mode Switch, J4 Display On, J5 Reset, J6 DHT22 innen, J7 DHT22 außen, J8 Display, J9 Door Open Sens, U1 Tiny_RTC_DS1307

Commit message: Added functionality to reset (power off/on) sensors on startup; Updated Schmatics
Connections:
- net +5V: now also R2.2; no longer J6.1 (Pin_1), J7.1 (Pin_1), R2.1
- net at A1.8 (D5), J6.2 (Pin_2): now also R2.1; no longer R2.2
- net at A1.11 (D8): now also J6.1 (Pin_1), J7.1 (Pin_1)
- no-connect marks 22 -> 21
Other:
- note added: "3.1"
- note removed: "3.0"
- moved on the sheet: R2, R3, R4

Commit message: Added feedback line from Relais-Input to D9 of Arduino. So it's possible to read back the current van state even if the arduino output signal is overridden by the mode switch.
Connections:
- net at J3.2 (Pin_2), R1.2, RLY1.1 (switch): now also A1.12 (D9)
- no-connect marks 21 -> 20
Changed lines of the file:
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@@
   (junction (at 208.915 132.08) (diameter 0) (color 0 0 0 0)
+  )
+  (junction (at 87.63 59.055) (diameter 0) (color 0 0 0 0)
   )
   (junction (at 87.63 57.785) (diameter 0) (color 0 0 0 0)
@@
   (no_connect (at 164.465 109.22))
   (no_connect (at 228.6 83.82))
-  (no_connect (at 139.065 101.6))
   (wire (pts (xy 208.915 129.54) (xy 208.915 127))
     (stroke (width 0) (type default) (color 0 0 0 0))
@@
     (stroke (width 0) (type default) (color 0 0 0 0))
   )
+  (wire (pts (xy 123.825 101.6) (xy 123.825 59.055))
+    (stroke (width 0) (type default) (color 0 0 0 0))
+  )
   (wire (pts (xy 75.565 83.82) (xy 139.065 83.82))
     (stroke (width 0) (type default) (color 0 0 0 0))
@@
     (stroke (width 0) (type default) (color 0 0 0 0))
   )
-  (wire (pts (xy 87.63 57.785) (xy 87.63 66.04))
+  (wire (pts (xy 139.065 101.6) (xy 123.825 101.6))
+    (stroke (width 0) (type default) (color 0 0 0 0))
+  )
+  (wire (pts (xy 87.63 57.785) (xy 87.63 59.055))
     (stroke (width 0) (type default) (color 0 0 0 0))
   )
@@
     (stroke (width 0) (type default) (color 0 0 0 0))
   )
+  (wire (pts (xy 87.63 59.055) (xy 123.825 59.055))
+    (stroke (width 0) (type default) (color 0 0 0 0))
+  )
   (wire (pts (xy 154.305 47.625) (xy 154.305 41.275))
     (stroke (width 0) (type default) (color 0 0 0 0))
@@
     (stroke (width 0) (type default) (color 0 0 0 0))
   )
+  (wire (pts (xy 87.63 59.055) (xy 87.63 66.04))
+    (stroke (width 0) (type default) (color 0 0 0 0))
+  )
